File: Schematics/Teensy_v1.3.sch (EAGLE design)
At the start: 10 parts, among them IC5 SN, IC6 YM, IC7 7.68MHz, IC8 3.57MHz, J1 OLED_128X64_I2C, J3 POWER_JACK

Commit message: Total Resdesign
This should probably be considered a 2.0 rev
Parts:
- added C1: 10uF, resistor:CPOL-USE2-5
- added C2: 100nF, resistor:C-EU025-025X050
- added IC1: LD117AV33, v-reg:LD117AV33
- added J2: HC-06, SparkFun-Connectors:CONN_04
Connections:
- net NEXT_BUTTON renamed BUTTON4
- net RAND_BUTTON renamed BUTTON3
- removed net 3V3: J1.1, U$1.3.3V
- removed net PAUSE: SV1.2, U$1.20/A6/PWM
- removed net PREV_BUTTON: SV1.1, U$1.21/A7/PWM
- new net BUTTON1: SV1.1, U$1.20/A6/PWM
- new net BUTTON2: SV1.2, U$1.21/A7/PWM
- new net N$14: C5.1
- new net N$16: C1.-
- new net N$17: C2.-
- new net N$18: C5.2
- new net N$3: IC1.OUT, J3.PWR, U$7.P$2
- new net N$5: IC1.BYPASS
- new net N$7: IC1.+IN
- new net RX: J2.3, U$1.10/TX2/PWM
- new net TX: J2.4, U$1.9/RX2/PWM
- new net VCC: C1.+, IC1.OUT, J1.1
- net 5V: now also C2.2, IC1.IN, IC1.VS, J2.1, U$7.P$1; no longer U$7.P$2
- net GND: now also C1.-, C2.1, IC1.-IN, IC1.ADJ, IC1.GND, J2.2, J2.S, J3.GNDBREAK
- net N$2: no longer J3.PWR, U$7.P$1
- net N$20: now also J2.T
- net N$21: now also J2.R
- net YM_MOL: now also C2.+
- net YM_MOR: now also C1.+
Other:
- note added: "OLED SCREEN AND REGULATOR"
- note added: "To Audio Output"
- note added: "UART BT"
- moved on the sheet: C5, IC5, IC6, IC7, IC8, J1, J3, SV1, U$1, U$7
